Commit message: feat(assets): swap the Dex3-1 hands for passive rubber ones
The hardware has rubber hands, and the depth cameras must see the meshes the
hardware has -- self-scanning is why this is more than cosmetic.

Three edits per side, in swap_rubber_hands():
  - delete the eight Dex3 links and their fixed joints;
  - restore wrist_yaw's inertial from the UNMERGED g1_21j_29dof.urdf;
  - weld the rubber hand on at the Dex3's own *_hand_palm_joint origin.

Step two is the one that bites. Our base asset merged the whole Dex3 into
wrist_yaw (0.084576 -> 0.781122 kg) and left the 16 finger links as 1 ug visual
carriers, so bolting a 0.170 kg hand on without restoring the bare wrist would
double-count 0.70 kg per side. The builder refuses unless merged-minus-bare
equals the Dex3 links' mass in the unmerged source, so a base asset that merges
something else into that wrist says so rather than losing the mass silently.

Numbers are from upstream g1_29dof_mode_11.urdf -- the variant this robot is, so
the hand comes from the same file as the motor specs. Verified three ways, which
would have to fail together: that file's left_wrist_yaw_link inertial is
byte-identical to ours in all eight fields; the mount is the Dex3's own palm-joint
origin, which our source states independently; and left_rubber_hand.STL is
watertight at 159.75 cm^3, so 0.170 kg implies 1064 kg/m^3 and that mesh's
uniform-density tensor reproduces all six upstream inertia terms to within 6%.

Verified after the swap: no dangling link references; the 29 actuated joints
identical in name AND order; every one of the 30 shared non-hand link frames
unmoved to 0.000000 mm. Links 53 -> 39, joints 52 -> 38. Robot 36.168 -> 37.755 kg
(-1.053 hands, +2.640 payload); CoM (9.4, 0.0, -54.7) mm vs the base's
(27.7, 0.1, -66.4).

No <collision> on the hands -- upstream gives them none and neither did the Dex3.

Two things this arms for the USD/MJCF regen, neither live yet:
  - features.HAND_FRAMES names left/right_palm_link, which the MJCF carries as
    bodies at the identical mount. Generating the MJCF from this URDF renames them
    to *_rubber_hand and FKChain will raise "end-effector frame not a body".
  - g1_self_scan.HAND_LINKS is the 8-per-side pattern and test_g1_self_scan pins
    len(SELF_SCAN_LINKS) == 26 + 16.

Co-Authored-By: Claude Opus 5 (1M context) <noreply@anthropic.com>

File: robot_assets/g1_perceptive/g1_perceptive.urdf (robot description, URDF)
Before this commit: robot g1_21j, 53 links, 52 joints
Links:
- removed link left_hand_index_0_link
- removed link left_hand_index_1_link
- removed link left_hand_middle_0_link
- removed link left_hand_middle_1_link
- removed link left_hand_palm_link
- removed link left_hand_thumb_0_link
- removed link left_hand_thumb_1_link
- removed link left_hand_thumb_2_link
- removed link right_hand_index_0_link
- removed link right_hand_index_1_link
- removed link right_hand_middle_0_link
- removed link right_hand_middle_1_link
- removed link right_hand_palm_link
- removed link right_hand_thumb_0_link
- removed link right_hand_thumb_1_link
- removed link right_hand_thumb_2_link
- added link left_rubber_hand, mass 0.17; visual mesh filename=../g1/g1_21j/meshes/left_rubber_hand.STL
- added link right_rubber_hand, mass 0.17; visual mesh filename=../g1/g1_21j/meshes/right_rubber_hand.STL
- link left_wrist_yaw_link: mass 0.78112246 -> 0.08457647
- link right_wrist_yaw_link: mass 0.78112246 -> 0.08457647
Joints:
- removed joint left_hand_index_0_link_fixed_joint
- removed joint left_hand_index_1_link_fixed_joint
- removed joint left_hand_middle_0_link_fixed_joint
- removed joint left_hand_middle_1_link_fixed_joint
- removed joint left_hand_palm_link_fixed_joint
- removed joint left_hand_thumb_0_link_fixed_joint
- removed joint left_hand_thumb_1_link_fixed_joint
- removed joint left_hand_thumb_2_link_fixed_joint
- removed joint right_hand_index_0_link_fixed_joint
- removed joint right_hand_index_1_link_fixed_joint
- removed joint right_hand_middle_0_link_fixed_joint
- removed joint right_hand_middle_1_link_fixed_joint
- removed joint right_hand_palm_link_fixed_joint
- removed joint right_hand_thumb_0_link_fixed_joint
- removed joint right_hand_thumb_1_link_fixed_joint
- removed joint right_hand_thumb_2_link_fixed_joint
- added joint left_hand_palm_joint: type fixed, parent left_wrist_yaw_link, child left_rubber_hand, origin xyz=0.0415 0.003 0 rpy=0 0 0
- added joint right_hand_palm_joint: type fixed, parent right_wrist_yaw_link, child right_rubber_hand, origin xyz=0.0415 -0.003 0 rpy=0 0 0

Commit message: feat(assets): apply the mode_11 deltas, and derive the merged asset from them
mode_11 is the variant this robot IS -- high-torque hip (22.5 gear), revolute-35
waist, light wrists. Our source predated it. Motors, waist geometry and the hands
land in one patch because they force one retrain between them.

The merge recipe was NOT lost, which Part 1.1 assumed it was: merge_urdf_joints.py
with no --keep reproduces the shipped g1_21j_box_merged_29j.urdf exactly -- 30
links, 29 joints, zero difference in mass, CoM, inertia, joint frames or limits. So
the box foot collider, the pelvis_link rename and the heel/toe frames survive a
re-derive because they live in the source already. The pipeline is now:

  g1_21j_29dof.urdf
    -> apply_mode11_deltas.py            g1_21j_29dof_mode11.urdf
    -> merge_urdf_joints.py --keep *_hand_palm_joint
                                         g1_21j_box_merged_29j_mode11.urdf
    -> make_perceptive_urdf.py           g1_perceptive.urdf

reference/g1_29dof_mode_11.urdf is vendored (sha recorded, BSD-3) so the patch reads
its VALUES from a file under version control. What is written down is only the
SCOPE, because a blind sync would revert our local customisations; the reference
README lists them.

Applied: 25 joint limits, 6 joint frames, 3 link inertials, 16 links out / 2 in.
The waist chain drops the torso 10 mm and the shoulder, logo and head mounts each
rise 10 mm inside it, so 28 of 30 shared link frames do not move at all -- the arms
are physically where they were. Robot 36.168 -> 33.342 kg, and 35.982 with payload.

The mass post-condition earns its place: it fired on the first run over 2 ug,
because I had transcribed the Dex3 mass with a 1 ug rounding. expected_delta_kg()
now derives both sides from the same two files and it closes at -2.826091980 with a
1 ng tolerance. It is deliberately not the two totals' difference -- upstream also
dropped two 1 g visual tokens we keep and added sensor frames we do not take.

Doing the hands here deletes the un-merge step make_perceptive_urdf.py needed a
commit ago: the merge folded the Dex3 into wrist_yaw, so swapping afterwards meant
subtracting 0.70 kg a side back out. With --keep on the palm joints it never gets
folded in. That file is now purely what we bolted on.

Actuators (Part 1.4). Hip pitch moves to the 22.5 gain class WITH its effort limit,
which is the whole trap: G1_ACTION_SCALE is 0.125 * effort / stiffness, so moving
the limit alone would have grown the hip-pitch action range to 0.4324 instead of
shrinking it to 0.1753. Ankles and waist roll/pitch 50 -> 35 N*m, both 0.700x.
Two beyond the plan's table, found by reading the real file: waist_yaw velocity was
37 and mode_11 says 32, and the wrists needed a velocity DICT -- they shared one
scalar 37, but roll is arm-class and pitch/yaw are the light motors at 22 rad/s.

EFFORT_OVERRIDES_URDF is now empty. It carried hip roll, where our URDF said 88 and
the cfg 139; the URDF was the stale side and the patch reconciled it.

test_velocity_limits_come_from_the_cfg_not_the_urdf was a Part 0 pin -- the old URDF
had a blanket 12 rad/s no motor has, so the two could not be compared, and its own
docstring said to convert it if they ever became real. They have, so it now compares
joint for joint and the third copy of these numbers has a guard.

train.py prints the resolved table at start, same reason the FM trainer prints its
exteroception band: the action scale is derived, so a gear change rescales the
policy silently and no runtime output would show it.

1137 tests pass.

Co-Authored-By: Claude Opus 5 (1M context) <noreply@anthropic.com>

File: robot_assets/g1_perceptive/g1_perceptive.urdf (robot description, URDF)
Before this commit: robot g1_21j, 39 links, 38 joints
Links:
- link left_rubber_hand: mass 0.17 -> 0.170
- link right_rubber_hand: mass 0.17 -> 0.170
- link torso_link: mass 9.6 -> 7.818
- link waist_roll_link: mass 0.047 -> 0.086
- link waist_yaw_link: mass 0.244 -> 0.214
Joints:
- joint left_ankle_pitch_joint: limit lower=-0.87267 upper=0.5236 effort=50 velocity=12 -> lower=-0.87267 upper=0.5236 effort=35 velocity=30
- joint left_ankle_roll_joint: limit lower=-0.2618 upper=0.2618 effort=50 velocity=12 -> lower=-0.2618 upper=0.2618 effort=35 velocity=30
- joint left_elbow_joint: limit lower=-1.0472 upper=2.0944 effort=25 velocity=12 -> lower=-1.0472 upper=2.0944 effort=25 velocity=37
- joint left_hip_pitch_joint: limit lower=-2.5307 upper=2.8798 effort=88 velocity=12 -> lower=-2.5307 upper=2.8798 effort=139 velocity=20
- joint left_hip_roll_joint: limit lower=-0.5236 upper=2.9671 effort=88 velocity=12 -> lower=-0.5236 upper=2.9671 effort=139 velocity=20
- joint left_hip_yaw_joint: limit lower=-2.7576 upper=2.7576 effort=88 velocity=12 -> lower=-2.7576 upper=2.7576 effort=88 velocity=32
- joint left_knee_joint: limit lower=-0.087267 upper=2.8798 effort=139 velocity=12 -> lower=-0.087267 upper=2.8798 effort=139 velocity=20
- joint left_shoulder_pitch_joint: limit lower=-3.0892 upper=2.6704 effort=25 velocity=12 -> lower=-3.0892 upper=2.6704 effort=25 velocity=37; origin xyz=0.0039563 0.10022 0.23778 rpy=0.27931 5.4949E-05 -0.00019159 -> xyz=0.0039563 0.10022 0.24778 rpy=0.27931 5.4949E-05 -0.00019159
- joint left_shoulder_roll_joint: limit lower=-1.5882 upper=2.2515 effort=25 velocity=12 -> lower=-1.5882 upper=2.2515 effort=25 velocity=37
- joint left_shoulder_yaw_joint: limit lower=-2.618 upper=2.618 effort=25 velocity=12 -> lower=-2.618 upper=2.618 effort=25 velocity=37
- joint left_wrist_roll_joint: limit lower=-1.972222054 upper=1.972222054 effort=25 velocity=12 -> lower=-1.972222054 upper=1.972222054 effort=25 velocity=37
- joint right_ankle_pitch_joint: limit lower=-0.87267 upper=0.5236 effort=50 velocity=12 -> lower=-0.87267 upper=0.5236 effort=35 velocity=30
- joint right_ankle_roll_joint: limit lower=-0.2618 upper=0.2618 effort=50 velocity=12 -> lower=-0.2618 upper=0.2618 effort=35 velocity=30
- joint right_elbow_joint: limit lower=-1.0472 upper=2.0944 effort=25 velocity=12 -> lower=-1.0472 upper=2.0944 effort=25 velocity=37
- joint right_hip_pitch_joint: limit lower=-2.5307 upper=2.8798 effort=88 velocity=12 -> lower=-2.5307 upper=2.8798 effort=139 velocity=20
- joint right_hip_roll_joint: limit lower=-2.9671 upper=0.5236 effort=88 velocity=12 -> lower=-2.9671 upper=0.5236 effort=139 velocity=20
- joint right_hip_yaw_joint: limit lower=-2.7576 upper=2.7576 effort=88 velocity=12 -> lower=-2.7576 upper=2.7576 effort=88 velocity=32
- joint right_knee_joint: limit lower=-0.087267 upper=2.8798 effort=139 velocity=12 -> lower=-0.087267 upper=2.8798 effort=139 velocity=20
- joint right_shoulder_pitch_joint: limit lower=-3.0892 upper=2.6704 effort=25 velocity=12 -> lower=-3.0892 upper=2.6704 effort=25 velocity=37; origin xyz=0.0039563 -0.10021 0.23778 rpy=-0.27931 5.4949E-05 0.00019159 -> xyz=0.0039563 -0.10021 0.24778 rpy=-0.27931 5.4949E-05 0.00019159
- joint right_shoulder_roll_joint: limit lower=-2.2515 upper=1.5882 effort=25 velocity=12 -> lower=-2.2515 upper=1.5882 effort=25 velocity=37
- joint right_shoulder_yaw_joint: limit lower=-2.618 upper=2.618 effort=25 velocity=12 -> lower=-2.618 upper=2.618 effort=25 velocity=37
- joint right_wrist_roll_joint: limit lower=-1.972222054 upper=1.972222054 effort=25 velocity=12 -> lower=-1.972222054 upper=1.972222054 effort=25 velocity=37
- joint waist_pitch_joint: limit lower=-0.52 upper=0.52 effort=50 velocity=12 -> lower=-0.52 upper=0.52 effort=35 velocity=30; origin xyz=0 0 0.019 rpy=0 0 0 -> xyz=0 0 0 rpy=0 0 0
- joint waist_roll_joint: limit lower=-0.52 upper=0.52 effort=50 velocity=12 -> lower=-0.52 upper=0.52 effort=35 velocity=30; origin xyz=-0.0039635 0 0.035 rpy=0 0 0 -> xyz=-0.0039635 0 0.044 rpy=0 0 0
- joint waist_yaw_joint: limit lower=-2.618 upper=2.618 effort=88 velocity=12 -> lower=-2.618 upper=2.618 effort=88 velocity=32

Commit message: feat(env): give the backpack a collider, DR and a contact sensor
Part 1.2's leftovers. The 2.64 kg pack had no randomisation, nothing watching it
for contact, and nothing it could collide with.

  add_torso_mass  now also scales backpack_thor_link and backpack_zed_link. Scoped
                  to torso_link, the largest new mass on the robot got no DR at all,
                  and its numbers are the least certain here -- weighed, with
                  "everything else" lumped into the Thor.
  backpack_com    new, +/-2 cm. Separate from torso_com because the uncertainty has a
                  different shape: where a bolt-on assembly actually ended up, plus
                  the plate and cabling whose spread is not in the inertia tensor
                  (that is the Thor BLOCK alone).
  backpack_contact  new. torso_contact matches the torso body exactly with no
                  trailing /.*, deliberately, so it does not cover a child link.

THE COLLIDER, and the bug it caused. A contact sensor on a body with no collider is
silently dead -- which is what torso_contact has been, since the torso box lives on
waist_yaw_link. So the shell got a box collider, and sized to its own mesh bbox it
overlapped the torso box by 2.09 mm across a 180 x 190 mm face. The two are rigidly
welded, so PhysX cannot resolve that by separating them; it just pushes. Measured in
a spawn-and-settle test: the robot drifted +0.38 m FORWARD in one second, when its
own added mass should carry it backwards -- and did, -0.19 m, before the collider
existed. Nothing failed and nothing warned.

Pulling the front face back 12.1 mm restores 10 mm of clearance, and the settle
trajectory becomes bit-identical to the no-collider run: root [-0.1892, 0.0026,
0.7237]. Nothing filters that pair -- PhysX only auto-filters ADJACENT links and
these are two joints apart -- so clearance is the mechanism, and
test_collider_geometry.py fails if any pair closes to under 2 mm at the rest pose.

A SECOND silent failure, found by the first fix. Adding the collision changed the
converter's output for that link: a link with both a visual and a collision gets an
inner geometry Xform, named after the VISUAL, falling back to the MESH FILENAME when
the visual is unnamed. Every stock G1 mesh is called after its link, so the fallback
looks like a rule -- until ASSY_backpack.STL lands under backpack_shell_link and the
prim comes out "ASSY_backpack". g1_self_scan builds targets from LINK names, so the
target named a prim that does not exist, which MultiMeshRayCaster reports as a log
line rather than an error: the pack would simply be missing from every depth image.
make_perceptive_urdf.py now names every visual after its link.

That also moved the shell between the two prim conventions, so it leaves _LEAF_LINKS
-- it is childless but has a collider, which is enough for the inner wrapper. The
comment now says what actually drives the doubling instead of "has child links".

Verified in sim: 39 bodies, 29 joints, 35.9821 kg matching the URDF, no zero-mass
bodies, finite after 1 s of settling. 1119 tests pass.

Co-Authored-By: Claude Opus 5 (1M context) <noreply@anthropic.com>

File: robot_assets/g1_perceptive/g1_perceptive.urdf (robot description, URDF)
Before this commit: robot g1_21j, 39 links, 38 joints
Links:
- link backpack_shell_link: geometry collision box size=0.15401 0.18748 0.25307; visual mesh filename=meshes/ASSY_backpack.STL
