Commit message: fix(assets): put the torso collider on the torso
The box lived on waist_yaw_link. Two consequences, both silent.

Waist roll and pitch are UNLOCKED on the 29-DOF robot (+/-0.52 rad) and
waist_yaw_link only yaws, so leaning the torso 30 degrees left its collider
standing upright in the wrong place.

And torso_contact names torso_link, which had no <collision> at all -- so one of
the five undesired_contacts sensors has never been able to fire, from the day the
waist was un-merged. A contact sensor on a collider-less body is not an error; it is
just permanently quiet.

Same box, re-expressed in the torso frame (origin 0.3 -> 0.246, x 0 -> 0.0039635) so
it does not move at zero joints. The spawn-and-settle trajectory is bit-identical to
before the move: root [-0.1892, 0.0026, 0.7237]. It does end up 10 mm lower in the
pelvis frame, because mode_11 drops the torso by that much and the shell now follows
the torso, which is the point.

It also REDUCES self-collision exposure: the arms and the backpack are children of
torso_link, so PhysX filters them against this box, where against waist_yaw_link
they were two joints away and unfiltered.

Edited as text, not via ElementTree: a round-trip through ET.indent reformatted 301
lines of blank space in a hand-maintained datum. And the comment says "plus or minus"
rather than using a double hyphen, because XML forbids one inside a comment -- the
first attempt broke the parse, which is the same rule CLAUDE.md records for MJCF.

test_collider_geometry.py grows a per-sensor check. It distinguishes an EXACT match
from a subtree match, which matters: left_hip_pitch_link has no collider of its own
and left_thigh_contact is fine because it watches ".../left_hip_pitch_link/.*". A
first version conflated the two and reported the knees and hips as dead sensors when
they are not.

1129 tests pass.

Co-Authored-By: Claude Opus 5 (1M context) <noreply@anthropic.com>

File: robot_assets/g1/g1_21j/g1_21j_29dof.urdf (robot description, URDF)
Before this commit: robot g1_21j, 64 links, 63 joints
Links:
- link torso_link: geometry collision box size=0.12 0.175 0.4; visual mesh filename=meshes/torso_link.STL
- link waist_yaw_link: geometry visual mesh filename=meshes/waist_yaw_link.STL

File: robot_assets/g1/g1_21j/g1_21j_29dof_mode11.urdf (robot description, URDF)
Before this commit: robot g1_21j, 50 links, 49 joints
Links:
- link torso_link: geometry collision box size=0.12 0.175 0.4; visual mesh filename=meshes/torso_link.STL
- link waist_yaw_link: geometry visual mesh filename=meshes/waist_yaw_link.STL

File: robot_assets/g1/g1_21j/g1_21j_box_merged_29j_mode11.urdf (robot description, URDF)
Before this commit: robot g1_21j, 32 links, 31 joints
Links:
- link torso_link: geometry collision box size=0.12 0.175 0.4; visual mesh filename=meshes/head_link.STL
- link waist_yaw_link: geometry visual mesh filename=meshes/waist_yaw_link.STL

File: robot_assets/g1_perceptive/g1_perceptive.urdf (robot description, URDF)
Before this commit: robot g1_21j, 39 links, 38 joints
Links:
- link torso_link: geometry collision box size=0.12 0.175 0.4; visual mesh filename=../g1/g1_21j/meshes/head_link.STL
- link waist_yaw_link: geometry visual mesh filename=../g1/g1_21j/meshes/waist_yaw_link.STL
